File: examples/03_LCD_16x2_AND_20x4/KiCad_Schematic/LCD.kicad_sch (KiCad schematic)
At the start: 12 parts, among them J1 KIT DIY 5~7W QN8066, U1 LCD 16x02 or 20x04

Commit message: DOc
Parts:
- added U2: Step Up 3.7V to 5V, Package_TO_SOT_SMD:SOT-23-6, symbol Regulator_Switching:MCP1640CCH
Connections:
- net +5V: now also U2.5 (VOUT); no longer J1.5 (Pin_5)
- net GND: now also U2.2 (GND)
- new net: J1.5 (Pin_5), U2.6 (VIN)
Other:
- note added: "3.7V"
Changed lines of the file:
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@@
   (junction (at 146.05 60.96) (diameter 0) (color 0 0 0 0)
   )
+  (junction (at 34.29 88.9) (diameter 0) (color 0 0 0 0)
+  )
   (junction (at 19.05 39.37) (diameter 0) (color 0 0 0 0)
   )
@@
     (stroke (width 0) (type default))
   )
+  (wire (pts (xy 35.56 93.98) (xy 20.32 93.98))
+    (stroke (width 0) (type default))
+  )
+  (wire (pts (xy 22.86 57.15) (xy 22.86 59.69))
+    (stroke (width 0) (type default))
+  )
   (wire (pts (xy 87.63 93.98) (xy 45.72 93.98))
     (stroke (width 0) (type default))
@@
     (stroke (width 0) (type default))
   )
+  (wire (pts (xy 19.05 39.37) (xy 19.05 41.91))
+    (stroke (width 0) (type default))
+  )
   (wire (pts (xy 83.82 52.07) (xy 135.89 52.07))
     (stroke (width 0) (type default))
   )
+  (wire (pts (xy 34.29 88.9) (xy 33.02 88.9))
+    (stroke (width 0) (type default))
+  )
   (wire (pts (xy 83.82 31.75) (xy 86.36 31.75))
     (stroke (width 0) (type default))
   )
-  (wire (pts (xy 35.56 93.98) (xy 35.56 92.71))
-    (stroke (width 0) (type default))
-  )
   (wire (pts (xy 123.19 39.37) (xy 83.82 39.37))
     (stroke (width 0) (type default))
@@
     (stroke (width 0) (type default))
   )
-  (wire (pts (xy 38.1 88.9) (xy 33.02 88.9))
+  (wire (pts (xy 38.1 88.9) (xy 34.29 88.9))
     (stroke (width 0) (type default))
   )
@@
     (stroke (width 0) (type default))
   )
+  (wire (pts (xy 33.02 69.85) (xy 34.29 69.85))
+    (stroke (width 0) (type default))
+  )
   (wire (pts (xy 87.63 41.91) (xy 87.63 93.98))
     (stroke (width 0) (type default))
@@
     (stroke (width 0) (type default))
   )
+  (wire (pts (xy 20.32 93.98) (xy 20.32 80.01))
+    (stroke (width 0) (type default))
+  )
   (wire (pts (xy 156.21 24.13) (xy 166.37 24.13))
     (stroke (width 0) (type default))
   )
-  (wire (pts (xy 35.56 92.71) (xy 33.02 92.71))
+  (wire (pts (xy 34.29 69.85) (xy 34.29 88.9))
     (stroke (width 0) (type default))
   )
@@
     (stroke (width 0) (type default))
   )
+  (wire (pts (xy 43.18 36.83) (xy 43.18 93.98))
+    (stroke (width 0) (type default))
+  )
+  (wire (pts (xy 40.64 39.37) (xy 44.45 39.37))
+    (stroke (width 0) (type default))
+  )
+  (wire (pts (xy 146.05 60.96) (xy 156.21 60.96))
+    (stroke (width 0) (type default))
+  )
+  (wire (pts (xy 161.29 46.99) (xy 161.29 50.8))
+    (stroke (width 0) (type default))
+  )
   (wire (pts (xy 19.05 36.83) (xy 19.05 39.37))
-    (stroke (width 0) (type default))
-  )
-  (wire (pts (xy 43.18 36.83) (xy 43.18 93.98))
-    (stroke (width 0) (type default))
-  )
-  (wire (pts (xy 40.64 39.37) (xy 44.45 39.37))
-    (stroke (width 0) (type default))
-  )
-  (wire (pts (xy 146.05 60.96) (xy 156.21 60.96))
-    (stroke (width 0) (type default))
-  )
-  (wire (pts (xy 161.29 46.99) (xy 161.29 50.8))
-    (stroke (width 0) (type default))
-  )
-  (wire (pts (xy 19.05 39.37) (xy 19.05 45.72))
     (stroke (width 0) (type default))
   )
@@
     (effects (font (size 1.27 1.27)) (justify right bottom))
   )
+  (text "3.7V" (at 24.13 96.52 0)
+    (effects (font (size 1.27 1.27)) (justify left bottom))
+  )
   (text "R1, R2, R3, and R4 are optional.\nHowever, consider using them to \nimprove the stability of the I2C \nbus and mitigate noise."
     (at 21.59 27.94 0)
@@
         (path "/03b4fd1c-f30e-47c7-82cf-518aad4befbb"
           (reference "#PWR06") (unit 1)
+        )
+      )
+    )
+  )
+  (symbol (lib_id "Regulator_Switching:MCP1640CCH") (at 25.4 69.85 90) (unit 1)
+    (in_bom yes) (on_board yes) (dnp no)
+    (property "Reference" "U2" (at 16.51 68.58 90)
+      (effects (font (size 1.27 1.27)) (justify left) hide)
+    )
+    (property "Value" "Step Up  3.7V to 5V" (at 15.24 80.01 0)
+      (effects (font (size 1.27 1.27)) (justify left))
+    )
+    (property "Footprint" "Package_TO_SOT_SMD:SOT-23-6" (at 31.75 68.58 0)
+      (effects (font (size 1.27 1.27) italic) (justify left) hide)
+    )
+    (property "Datasheet" "http://ww1.microchip.com/downloads/en/DeviceDoc/20002234D.pdf" (at 13.97 76.2 0)
+      (effects (font (size 1.27 1.27)) hide)
+    )
+    (pin "1")
+    (pin "2")
+    (pin "3")
+    (pin "4")
+    (pin "5")
+    (pin "6")
+    (instances
+      (project "LCD"
+        (path "/03b4fd1c-f30e-47c7-82cf-518aad4befbb"
+          (reference "U2") (unit 1)
         )
       )
@@
     )
   )
-  (symbol (lib_id "power:+5V") (at 19.05 45.72 180) (unit 1)
+  (symbol (lib_id "power:+5V") (at 19.05 41.91 180) (unit 1)
     (in_bom yes) (on_board yes) (dnp no) (fields_autoplaced)
-    (property "Reference" "#PWR08" (at 19.05 41.91 0)
-      (effects (font (size 1.27 1.27)) hide)
-    )
-    (property "Value" "+5V" (at 19.05 50.8 0)
-      (effects (font (size 1.27 1.27)))
-    )
-    (property "Footprint" "" (at 19.05 45.72 0)
-      (effects (font (size 1.27 1.27)) hide)
-    )
-    (property "Datasheet" "" (at 19.05 45.72 0)
+    (property "Reference" "#PWR08" (at 19.05 38.1 0)
+      (effects (font (size 1.27 1.27)) hide)
+    )
+    (property "Value" "+5V" (at 19.05 46.99 0)
+      (effects (font (size 1.27 1.27)))
+    )
+    (property "Footprint" "" (at 19.05 41.91 0)
+      (effects (font (size 1.27 1.27)) hide)
+    )
+    (property "Datasheet" "" (at 19.05 41.91 0)
       (effects (font (size 1.27 1.27)) hide)
     )
@@
         (path "/03b4fd1c-f30e-47c7-82cf-518aad4befbb"
           (reference "#PWR08") (unit 1)
-        )
-      )
-    )
-  )
-  (symbol (lib_id "power:+5V") (at 33.02 92.71 90) (unit 1)
-    (in_bom yes) (on_board yes) (dnp no)
-    (property "Reference" "#PWR09" (at 36.83 92.71 0)
-      (effects (font (size 1.27 1.27)) hide)
-    )
-    (property "Value" "+5V" (at 30.48 96.52 0)
-      (effects (font (size 1.27 1.27)))
-    )
-    (property "Footprint" "" (at 33.02 92.71 0)
-      (effects (font (size 1.27 1.27)) hide)
-    )
-    (property "Datasheet" "" (at 33.02 92.71 0)
-      (effects (font (size 1.27 1.27)) hide)
-    )
-    (pin "1")
-    (instances
-      (project "LCD"
-        (path "/03b4fd1c-f30e-47c7-82cf-518aad4befbb"
-          (reference "#PWR09") (unit 1)
         )
       )
@@
         )
       )
+    )
+  )
+  (symbol (lib_id "power:+5V") (at 22.86 57.15 0) (unit 1)
+    (in_bom yes) (on_board yes) (dnp no) (fields_autoplaced)
+    (property "Reference" "#PWR09" (at 22.86 60.96 0)
+      (effects (font (size 1.27 1.27)) hide)
+    )
+    (property "Value" "+5V" (at 22.86 52.07 0)
+      (effects (font (size 1.27 1.27)))
+    )
+    (property "Footprint" "" (at 22.86 57.15 0)
+      (effects (font (size 1.27 1.27)) hide)
+    )
+    (property "Datasheet" "" (at 22.86 57.15 0)
+      (effects (font (size 1.27 1.27)) hide)
+    )
+    (pin "1")
+    (instances
+      (project "LCD"
+        (path "/03b4fd1c-f30e-47c7-82cf-518aad4befbb"
+          (reference "#PWR09") (unit 1)
+        )
+      )

Commit message: Doc
Parts:
- removed U2: Step Up 3.7V to 5V, Package_TO_SOT_SMD:SOT-23-6, symbol Regulator_Switching:MCP1640CCH
- added U2: L78L05_SO8, Package_SO:SOIC-8_3.9x4.9mm_P1.27mm, symbol Regulator_Linear:L78L05_SO8
Connections:
- net +5V: now also U2.1 (OUT)
- net GND: now also U2.2 (GND), U2.3 (GND), U2.6 (GND), U2.7 (GND)
- new net +12V: U2.8 (IN)
Other:
- note added: "From the TX board"
- note removed: "3.7V"
Changed lines of the file:
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@@
   (junction (at 146.05 60.96) (diameter 0) (color 0 0 0 0)
   )
-  (junction (at 34.29 88.9) (diameter 0) (color 0 0 0 0)
-  )
   (junction (at 19.05 39.37) (diameter 0) (color 0 0 0 0)
   )
@@
   (junction (at 120.65 95.25) (diameter 0) (color 0 0 0 0)
   )
+  (junction (at 73.66 77.47) (diameter 0) (color 0 0 0 0)
+  )
   (junction (at 133.35 95.25) (diameter 0) (color 0 0 0 0)
   )
@@
     (stroke (width 0) (type default))
   )
-  (wire (pts (xy 35.56 93.98) (xy 20.32 93.98))
-    (stroke (width 0) (type default))
-  )
-  (wire (pts (xy 22.86 57.15) (xy 22.86 59.69))
-    (stroke (width 0) (type default))
-  )
   (wire (pts (xy 87.63 93.98) (xy 45.72 93.98))
     (stroke (width 0) (type default))
   )
+  (wire (pts (xy 52.07 81.28) (xy 52.07 77.47))
+    (stroke (width 0) (type default))
+  )
   (wire (pts (xy 156.21 49.53) (xy 156.21 60.96))
     (stroke (width 0) (type default))
@@
     (stroke (width 0) (type default))
   )
+  (wire (pts (xy 73.66 77.47) (xy 73.66 82.55))
+    (stroke (width 0) (type default))
+  )
   (wire (pts (xy 95.25 36.83) (xy 83.82 36.83))
     (stroke (width 0) (type default))
@@
     (stroke (width 0) (type default))
   )
+  (wire (pts (xy 59.69 85.09) (xy 59.69 87.63))
+    (stroke (width 0) (type default))
+  )
   (wire (pts (xy 105.41 87.63) (xy 105.41 95.25))
     (stroke (width 0) (type default))
@@
     (stroke (width 0) (type default))
   )
-  (wire (pts (xy 34.29 88.9) (xy 33.02 88.9))
+  (wire (pts (xy 33.02 88.9) (xy 38.1 88.9))
     (stroke (width 0) (type default))
   )
@@
     (stroke (width 0) (type default))
   )
-  (wire (pts (xy 38.1 88.9) (xy 34.29 88.9))
-    (stroke (width 0) (type default))
-  )
   (wire (pts (xy 40.64 39.37) (xy 40.64 93.98))
     (stroke (width 0) (type default))
   )
-  (wire (pts (xy 33.02 69.85) (xy 34.29 69.85))
-    (stroke (width 0) (type default))
-  )
   (wire (pts (xy 87.63 41.91) (xy 87.63 93.98))
     (stroke (width 0) (type default))
@@
     (stroke (width 0) (type default))
   )
-  (wire (pts (xy 20.32 93.98) (xy 20.32 80.01))
-    (stroke (width 0) (type default))
-  )
   (wire (pts (xy 156.21 24.13) (xy 166.37 24.13))
     (stroke (width 0) (type default))
   )
-  (wire (pts (xy 34.29 69.85) (xy 34.29 88.9))
+  (wire (pts (xy 67.31 77.47) (xy 73.66 77.47))
     (stroke (width 0) (type default))
   )
@@
     )
   )
-  (text "SCL" (at 45.72 78.74 90)
+  (text "SCL" (at 45.72 72.39 90)
     (effects (font (size 1.27 1.27)) (justify right bottom))
-  )
-  (text "3.7V" (at 24.13 96.52 0)
-    (effects (font (size 1.27 1.27)) (justify left bottom))
   )
   (text "R1, R2, R3, and R4 are optional.\nHowever, consider using them to \nimprove the stability of the I2C \nbus and mitigate noise."
@@
     (effects (font (size 1.27 1.27)) (justify left bottom))
   )
-  (text "PWM" (at 46.99 87.63 90)
+  (text "PWM" (at 48.26 96.52 90)
     (effects (font (size 1.27 1.27)) (justify right bottom))
   )
-  (text "SDA" (at 39.37 78.74 90)
+  (text "SDA" (at 39.37 72.39 90)
     (effects (font (size 1.27 1.27)) (justify right bottom))
   )
   (text "TRANSMITTER" (at 34.29 109.22 0)
     (effects (font (size 1.27 1.27) (thickness 0.254) bold (color 255 73 85 1)) (justify left bottom))
+  )
+  (text "From the \nTX board" (at 48.26 92.71 0)
+    (effects (font (size 1.27 1.27)) (justify left bottom))
   )
   (symbol (lib_id "power:GND") (at 146.05 64.77 0) (unit 1)
@@
     )
   )
-  (symbol (lib_id "Regulator_Switching:MCP1640CCH") (at 25.4 69.85 90) (unit 1)
+  (symbol (lib_id "power:+5V") (at 73.66 82.55 180) (unit 1)
+    (in_bom yes) (on_board yes) (dnp no) (fields_autoplaced)
+    (property "Reference" "#PWR02" (at 73.66 78.74 0)
+      (effects (font (size 1.27 1.27)) hide)
+    )
+    (property "Value" "+5V" (at 73.66 87.63 0)
+      (effects (font (size 1.27 1.27)))
+    )
+    (property "Footprint" "" (at 73.66 82.55 0)
+      (effects (font (size 1.27 1.27)) hide)
+    )
+    (property "Datasheet" "" (at 73.66 82.55 0)
+      (effects (font (size 1.27 1.27)) hide)
+    )
+    (pin "1")
+    (instances
+      (project "LCD"
+        (path "/03b4fd1c-f30e-47c7-82cf-518aad4befbb"
+          (reference "#PWR02") (unit 1)
+        )
+      )
+    )
+  )
+  (symbol (lib_id "Regulator_Linear:L78L05_SO8") (at 59.69 77.47 0) (unit 1)
     (in_bom yes) (on_board yes) (dnp no)
-    (property "Reference" "U2" (at 16.51 68.58 90)
-      (effects (font (size 1.27 1.27)) (justify left) hide)
-    )
-    (property "Value" "Step Up  3.7V to 5V" (at 15.24 80.01 0)
-      (effects (font (size 1.27 1.27)) (justify left))
-    )
-    (property "Footprint" "Package_TO_SOT_SMD:SOT-23-6" (at 31.75 68.58 0)
-      (effects (font (size 1.27 1.27) italic) (justify left) hide)
-    )
-    (property "Datasheet" "http://ww1.microchip.com/downloads/en/DeviceDoc/20002234D.pdf" (at 13.97 76.2 0)
+    (property "Reference" "U2" (at 59.69 71.12 0)
+      (effects (font (size 1.27 1.27)) hide)
+    )
+    (property "Value" "L78L05_SO8" (at 53.34 73.66 0)
+      (effects (font (size 1.27 1.27)))
+    )
+    (property "Footprint" "Package_SO:SOIC-8_3.9x4.9mm_P1.27mm" (at 62.23 72.39 0)
+      (effects (font (size 1.27 1.27) italic) hide)
+    )
+    (property "Datasheet" "http://www.st.com/content/ccc/resource/technical/document/datasheet/15/55/e5/aa/23/5b/43/fd/CD00000446.pdf/files/CD00000446.pdf/jcr:content/translations/en.CD00000446.pdf" (at 64.77 77.47 0)
       (effects (font (size 1.27 1.27)) hide)
     )
@@
     (pin "5")
     (pin "6")
+    (pin "7")
+    (pin "8")
     (instances
       (project "LCD"
         (path "/03b4fd1c-f30e-47c7-82cf-518aad4befbb"
           (reference "U2") (unit 1)
-        )
-      )
-    )
-  )
-  (symbol (lib_id "power:+5V") (at 73.66 77.47 180) (unit 1)
-    (in_bom yes) (on_board yes) (dnp no) (fields_autoplaced)
-    (property "Reference" "#PWR02" (at 73.66 73.66 0)
-      (effects (font (size 1.27 1.27)) hide)
-    )
-    (property "Value" "+5V" (at 73.66 82.55 0)
-      (effects (font (size 1.27 1.27)))
-    )
-    (property "Footprint" "" (at 73.66 77.47 0)
-      (effects (font (size 1.27 1.27)) hide)
-    )
-    (property "Datasheet" "" (at 73.66 77.47 0)
-      (effects (font (size 1.27 1.27)) hide)
-    )
-    (pin "1")
-    (instances
-      (project "LCD"
-        (path "/03b4fd1c-f30e-47c7-82cf-518aad4befbb"
-          (reference "#PWR02") (unit 1)
         )
       )
@@
     )
   )
+  (symbol (lib_id "power:+12V") (at 52.07 81.28 180) (unit 1)
+    (in_bom yes) (on_board yes) (dnp no)
+    (property "Reference" "#PWR012" (at 52.07 77.47 0)
+      (effects (font (size 1.27 1.27)) hide)
+    )
+    (property "Value" "+12V" (at 52.07 86.36 0)
+      (effects (font (size 1.27 1.27)))
+    )
+    (property "Footprint" "" (at 52.07 81.28 0)
+      (effects (font (size 1.27 1.27)) hide)
+    )
+    (property "Datasheet" "" (at 52.07 81.28 0)
+      (effects (font (size 1.27 1.27)) hide)
+    )
+    (pin "1")
+    (instances
+      (project "LCD"
+        (path "/03b4fd1c-f30e-47c7-82cf-518aad4befbb"
+          (reference "#PWR012") (unit 1)
+        )
+      )
+    )
+  )
   (symbol (lib_id "power:+5V") (at 161.29 50.8 180) (unit 1)
     (in_bom yes) (on_board yes) (dnp no) (fields_autoplaced)
@@
     )
   )
-  (symbol (lib_id "power:+5V") (at 22.86 57.15 0) (unit 1)
-    (in_bom yes) (on_board yes) (dnp no) (fields_autoplaced)
-    (property "Reference" "#PWR09" (at 22.86 60.96 0)
-      (effects (font (size 1.27 1.27)) hide)
-    )
-    (property "Value" "+5V" (at 22.86 52.07 0)
-      (effects (font (size 1.27 1.27)))
-    )
-    (property "Footprint" "" (at 22.86 57.15 0)
-      (effects (font (size 1.27 1.27)) hide)
-    )
-    (property "Datasheet" "" (at 22.86 57.15 0)
-      (effects (font (size 1.27 1.27)) hide)
-    )
-    (pin "1")
-    (instances
-      (project "LCD"
-        (path "/03b4fd1c-f30e-47c7-82cf-518aad4befbb"
-          (reference "#PWR09") (unit 1)
-        )
-      )
-    )
-  )
   (symbol (lib_id "power:GND") (at 71.12 19.05 180) (unit 1)
     (in_bom yes) (on_board yes) (dnp no) (fields_autoplaced)
@@
         )
       )
+    )
+  )
+  (symbol (lib_id "power:GND") (at 59.69 87.63 0) (unit 1)
+    (in_bom yes) (on_board yes) (dnp no) (fields_autoplaced)
+    (property "Reference" "#PWR09" (at 59.69 93.98 0)
+      (effects (font (size 1.27 1.27)) hide)
+    )
+    (property "Value" "GND" (at 59.69 92.71 0)
+      (effects (font (size 1.27 1.27)))
+    )
+    (property "Footprint" "" (at 59.69 87.63 0)
+      (effects (font (size 1.27 1.27)) hide)
+    )
+    (property "Datasheet" "" (at 59.69 87.63 0)
+      (effects (font (size 1.27 1.27)) hide)
+    )
+    (pin "1")
+    (instances
+      (project "LCD"
+        (path "/03b4fd1c-f30e-47c7-82cf-518aad4befbb"
+          (reference "#PWR09") (unit 1)
+        )
+      )

Commit message: Doc
Parts:
- removed R1, R2: 10K, symbol Device:R
- removed R3, R4: 1K, symbol Device:R
- removed U2: L78L05_SO8, Package_SO:SOIC-8_3.9x4.9mm_P1.27mm, symbol Regulator_Linear:L78L05_SO8
- added U2: bidirectional I2C level shifter, symbol Interface:TCA9406DC
- added U3: Step Up 3.3V to 5V, Package_TO_SOT_SMD:SOT-23-6, symbol Regulator_Switching:MCP1640CCH
Connections:
- net +5V: now also U3.5 (VOUT)
- net GND: now also U3.2 (GND)
- net at J1.2 (Pin_2): now also U2.4 (SDA_A)
- net at J1.3 (Pin_3): now also U2.5 (SCL_A)
- net at J1.5 (Pin_5): now also U3.6 (VIN)
- net at A1.24 (A5): now also U2.8 (SCL_B)
- net at A1.23 (A4): now also U2.1 (SDA_B)
Other:
- note added: "To Arduino VIN"
- note removed: "From the TX board"
- moved on the sheet: A1, DOWN, MENU, RESET, RV1, UP

Commit message: Doc
Other:
- note added: "3.3V"
- note added: "5V"
Changed lines of the file:
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@@
     (effects (font (size 1.27 1.27)) (justify right bottom))
+  )
+  (text "3.3V" (at 72.39 73.66 0)
+    (effects (font (size 1.27 1.27)) (justify left bottom))
   )
   (text "SDA" (at 66.04 83.82 90)
     (effects (font (size 1.27 1.27)) (justify right bottom))
   )
+  (text "5V" (at 73.66 62.23 0)
+    (effects (font (size 1.27 1.27)) (justify left bottom))
+  )
   (text "TRANSMITTER" (at 60.96 134.62 0)
