File: examples/03_LCD_16x2_AND_20x4/KiCad_Schematic/Nano/LCD.kicad_sch (KiCad schematic)
At the start: 10 parts, among them J1 KIT DIY 5~7W QN8066, U1 LCD 16x02 or 20x04, U2 bidirectional I2C level shift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, U3 Step Up 3.3V to 5V

Commit message: Doc
Parts:
- removed RESET: ~, symbol Switch:SW_Push
Other:
- note removed: "R1, R2, R3, and R4 are optional. However, consider using them to improve the stability of the I2C bus and mitigate noise."
Changed lines of the file:
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@@
   (junction (at 147.32 96.52) (diameter 0) (color 0 0 0 0)
   )
-  (junction (at 160.02 96.52) (diameter 0) (color 0 0 0 0)
-  )
   (wire (pts (xy 196.85 21.59) (xy 196.85 19.05))
     (stroke (width 0) (type default))
@@
     (stroke (width 0) (type default))
   )
-  (wire (pts (xy 173.99 88.9) (xy 173.99 96.52))
-    (stroke (width 0) (type default))
-  )
   (wire (pts (xy 113.03 33.02) (xy 113.03 25.4))
     (stroke (width 0) (type default))
@@
     (stroke (width 0) (type default))
   )
-  (wire (pts (xy 163.83 58.42) (xy 110.49 58.42))
-    (stroke (width 0) (type default))
-  )
   (wire (pts (xy 110.49 35.56) (xy 115.57 35.56))
     (stroke (width 0) (type default))
@@
     (stroke (width 0) (type default))
   )
-  (wire (pts (xy 163.83 88.9) (xy 163.83 58.42))
-    (stroke (width 0) (type default))
-  )
   (wire (pts (xy 172.72 19.05) (xy 172.72 20.32))
     (stroke (width 0) (type default))
@@
   )
   (wire (pts (xy 113.03 25.4) (xy 162.56 25.4))
-    (stroke (width 0) (type default))
-  )
-  (wire (pts (xy 173.99 96.52) (xy 160.02 96.52))
     (stroke (width 0) (type default))
   )
@@
     (effects (font (size 1.27 1.27)) (justify left bottom))
   )
-  (text "R1, R2, R3, and R4 are optional.\nHowever, consider using them to \nimprove the stability of the I2C \nbus and mitigate noise."
-    (at 48.26 29.21 0)
-    (effects (font (size 1.27 1.27)) (justify left bottom))
-  )
   (text "PWM" (at 82.55 97.79 0)
     (effects (font (size 1.27 1.27)) (justify right bottom))
@@
         )
       )
-    )
-  )
-  (symbol (lib_id "Switch:SW_Push") (at 168.91 88.9 0) (unit 1)
-    (in_bom yes) (on_board yes) (dnp no) (fields_autoplaced)
-    (property "Reference" "RESET" (at 168.91 83.82 0)
-      (effects (font (size 1.27 1.27)))
-    )
-    (property "Value" "~" (at 168.91 83.82 0)
-      (effects (font (size 1.27 1.27)))
-    )
-    (property "Footprint" "" (at 168.91 83.82 0)
-      (effects (font (size 1.27 1.27)) hide)
-    )
-    (property "Datasheet" "~" (at 168.91 83.82 0)
-      (effects (font (size 1.27 1.27)) hide)
-    )
-    (pin "1")
-    (pin "2")
-    (instances
-      (project "LCD"
-        (path "/03b4fd1c-f30e-47c7-82cf-518aad4befbb"
-          (reference "RESET") (unit 1)
-        )
-      )

Commit message: Doc
Connections:
- net GND: now also U1.5 (R/~{W}); no longer U1.4 (RS)
- net at A1.15 (D12): now also U1.4 (RS); no longer U1.5 (R/~{W})
Changed lines of the file:
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@@
+    (stroke (width 0) (type default))
+  )
+  (wire (pts (xy 156.21 27.94) (xy 162.56 27.94))
     (stroke (width 0) (type default))
   )
@@
     (stroke (width 0) (type default))
   )
+  (wire (pts (xy 162.56 30.48) (xy 115.57 30.48))
+    (stroke (width 0) (type default))
+  )
   (wire (pts (xy 196.85 19.05) (xy 172.72 19.05))
     (stroke (width 0) (type default))
   )
+  (wire (pts (xy 115.57 30.48) (xy 115.57 35.56))
+    (stroke (width 0) (type default))
+  )
   (wire (pts (xy 44.45 78.74) (xy 44.45 81.28))
     (stroke (width 0) (type default))
@@
     (stroke (width 0) (type default))
   )
-  (wire (pts (xy 158.75 30.48) (xy 158.75 33.02))
-    (stroke (width 0) (type default))
-  )
   (wire (pts (xy 135.89 45.72) (xy 110.49 45.72))
     (stroke (width 0) (type default))
@@
     (stroke (width 0) (type default))
   )
-  (wire (pts (xy 110.49 35.56) (xy 115.57 35.56))
+  (wire (pts (xy 115.57 35.56) (xy 110.49 35.56))
     (stroke (width 0) (type default))
   )
@@
     (stroke (width 0) (type default))
   )
-  (wire (pts (xy 115.57 35.56) (xy 115.57 27.94))
-    (stroke (width 0) (type default))
-  )
-  (wire (pts (xy 162.56 30.48) (xy 158.75 30.48))
-    (stroke (width 0) (type default))
-  )
   (wire (pts (xy 196.85 29.21) (xy 196.85 33.02))
     (stroke (width 0) (type default))
@@
   )
   (wire (pts (xy 67.31 38.1) (xy 85.09 38.1))
-    (stroke (width 0) (type default))
-  )
-  (wire (pts (xy 115.57 27.94) (xy 162.56 27.94))
     (stroke (width 0) (type default))
   )
@@
     )
   )
-  (symbol (lib_id "power:GND") (at 158.75 33.02 0) (unit 1)
+  (symbol (lib_id "power:GND") (at 156.21 27.94 270) (unit 1)
     (in_bom yes) (on_board yes) (dnp no)
-    (property "Reference" "#PWR06" (at 158.75 39.37 0)
+    (property "Reference" "#PWR06" (at 149.86 27.94 0)
       (effects (font (size 1.27 1.27)) hide)
     )
-    (property "Value" "GND" (at 158.75 36.83 0)
+    (property "Value" "GND" (at 152.4 27.94 0)
       (effects (font (size 1.27 1.27)))
     )
-    (property "Footprint" "" (at 158.75 33.02 0)
+    (property "Footprint" "" (at 156.21 27.94 0)
       (effects (font (size 1.27 1.27)) hide)
     )
-    (property "Datasheet" "" (at 158.75 33.02 0)
+    (property "Datasheet" "" (at 156.21 27.94 0)
       (effects (font (size 1.27 1.27)) hide)
     )
