File: examples/03_LCD_16x2_AND_20x4/KiCad_Schematic/ProMini/LCD.kicad_sch (KiCad schematic)
At the start: 9 parts, among them J1 KIT DIY 5~7W QN8066, U1 LCD 16x02 or 20x04

Commit message: Doc
Connections:
- net GND: now also U1.5 (R/~{W}); no longer U1.4 (RS)
- net at A1.15 (D12): now also U1.4 (RS); no longer U1.5 (R/~{W})
Changed lines of the file:
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@@
+    (stroke (width 0) (type default))
+  )
+  (wire (pts (xy 162.56 30.48) (xy 115.57 30.48))
     (stroke (width 0) (type default))
   )
@@
     (stroke (width 0) (type default))
   )
-  (wire (pts (xy 158.75 30.48) (xy 158.75 33.02))
-    (stroke (width 0) (type default))
-  )
   (wire (pts (xy 135.89 45.72) (xy 110.49 45.72))
     (stroke (width 0) (type default))
@@
     (stroke (width 0) (type default))
   )
+  (wire (pts (xy 158.75 27.94) (xy 162.56 27.94))
+    (stroke (width 0) (type default))
+  )
   (wire (pts (xy 110.49 35.56) (xy 115.57 35.56))
     (stroke (width 0) (type default))
@@
     (stroke (width 0) (type default))
   )
-  (wire (pts (xy 115.57 35.56) (xy 115.57 27.94))
-    (stroke (width 0) (type default))
-  )
-  (wire (pts (xy 162.56 30.48) (xy 158.75 30.48))
+  (wire (pts (xy 115.57 30.48) (xy 115.57 35.56))
     (stroke (width 0) (type default))
   )
@@
   )
   (wire (pts (xy 67.31 38.1) (xy 85.09 38.1))
-    (stroke (width 0) (type default))
-  )
-  (wire (pts (xy 115.57 27.94) (xy 162.56 27.94))
     (stroke (width 0) (type default))
   )
@@
     )
   )
-  (symbol (lib_id "power:GND") (at 158.75 33.02 0) (unit 1)
+  (symbol (lib_id "power:GND") (at 158.75 27.94 270) (unit 1)
     (in_bom yes) (on_board yes) (dnp no)
-    (property "Reference" "#PWR06" (at 158.75 39.37 0)
+    (property "Reference" "#PWR06" (at 152.4 27.94 0)
       (effects (font (size 1.27 1.27)) hide)
     )
-    (property "Value" "GND" (at 158.75 36.83 0)
+    (property "Value" "GND" (at 154.94 27.94 0)
       (effects (font (size 1.27 1.27)))
     )
-    (property "Footprint" "" (at 158.75 33.02 0)
+    (property "Footprint" "" (at 158.75 27.94 0)
       (effects (font (size 1.27 1.27)) hide)
     )
-    (property "Datasheet" "" (at 158.75 33.02 0)
+    (property "Datasheet" "" (at 158.75 27.94 0)
       (effects (font (size 1.27 1.27)) hide)
     )

Commit message: Doc
Connections:
- net +3V3: now also U1.A2
Changed lines of the file:
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@@
+    (stroke (width 0) (type default))
+  )
+  (wire (pts (xy 182.88 48.26) (xy 194.31 48.26))
     (stroke (width 0) (type default))
   )
@@
     (stroke (width 0) (type default))
   )
+  (wire (pts (xy 194.31 48.26) (xy 194.31 49.53))
+    (stroke (width 0) (type default))
+  )
   (wire (pts (xy 110.49 35.56) (xy 115.57 35.56))
     (stroke (width 0) (type default))
@@
   )
   (wire (pts (xy 67.31 38.1) (xy 85.09 38.1))
-    (stroke (width 0) (type default))
-  )
-  (wire (pts (xy 182.88 48.26) (xy 187.96 48.26))
     (stroke (width 0) (type default))
   )
@@
     (effects (font (size 1.27 1.27) (thickness 0.254) bold (color 255 73 85 1)) (justify left bottom))
   )
+  (text "It is a version of 3.3V LCD16x02" (at 199.39 78.74 90)
+    (effects (font (size 1.27 1.27)) (justify left bottom))
+  )
   (text "Arduino Pro Mini VCC Pin" (at 87.63 81.28 0)
     (effects (font (size 1.27 1.27)) (justify left bottom))
@@
         )
       )
+    )
+  )
+  (symbol (lib_id "power:+3V3") (at 194.31 49.53 180) (unit 1)
+    (in_bom yes) (on_board yes) (dnp no) (fields_autoplaced)
+    (property "Reference" "#PWR08" (at 194.31 45.72 0)
+      (effects (font (size 1.27 1.27)) hide)
+    )
+    (property "Value" "+3V3" (at 194.31 54.61 0)
+      (effects (font (size 1.27 1.27)))
+    )
+    (property "Footprint" "" (at 194.31 49.53 0)
+      (effects (font (size 1.27 1.27)) hide)
+    )
+    (property "Datasheet" "" (at 194.31 49.53 0)
+      (effects (font (size 1.27 1.27)) hide)
+    )
+    (pin "1")
+    (instances
+      (project "LCD"
+        (path "/03b4fd1c-f30e-47c7-82cf-518aad4befbb"
+          (reference "#PWR08") (unit 1)
+        )
+      )
