File: examples/99_UNDER_CONSTRUCTION/03_LCD_16x2_AND_20x4/KiCad_Schematic/ProMini/LCD.kicad_sch (KiCad schematic)
At the start: 10 parts, among them J1 KIT DIY 5~7W QN8066, U1 LCD 16x02 or 20x04, U2 bidirectional I2C level shift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, U3 Step Up 3.3V to 5V

Commit message: Doc
Parts:
- removed RESET: ~, symbol Switch:SW_Push
- removed U2: bidirectional I2C level shifter, symbol Interface:TCA9406DC
- removed U3: Step Up 3.3V to 5V, Package_TO_SOT_SMD:SOT-23-6, symbol Regulator_Switching:MCP1640CCH
- added R1, R2: 10K, symbol Device:R
- A1: value Arduino_Nano_v3.x -> Arduino Pro Mini
Connections:
- net +5V is gone; now on net +3V3: A1.30 (VIN), RV1.1, U1.2 (VDD), U1.A2
- net GND: now also U1.5 (R/~{W}); no longer U1.4 (RS)
- net at J1.2 (Pin_2): now also A1.23 (A4), R1.2
- net at J1.3 (Pin_3): now also A1.24 (A5), R2.2
- net +3V3: now reaches J1.5 (Pin_5)
- net +3V3: now also R1.1, R2.1
- net at A1.15 (D12): now also U1.4 (RS); no longer U1.5 (R/~{W})
Other:
- note added: "Arduino Pro Mini"
- note added: "Arduino Pro Mini VCC Pin"
- note added: "It is a version of 3.3V LCD16x02"
- note added: "R1 and R2 can improve the I2C communication."
- note removed: "3.3V"
- note removed: "5V"
- note removed: "R1, R2, R3, and R4 are optional. However, consider using them to improve the stability of the I2C bus and mitigate noise."
- note removed: "To Arduino VIN"
- title: QN8066 FM TRANSMITTER - LCD16X2 OR LCD20X4 -> QN8066 FM TRANSMITTER - Arduino Pro Mini and LCD
