File: examples/03_LCD_16x2_AND_20x4/KiCad_Schematic/ESP32/ESP32_LCD_ENCODER/ESP32_LCD_ENCODER.kicad_sch (KiCad schematic)
At the start: 3 parts, among them SW1 ENCODER, U2 LCD16X2

Commit message: Doc
Parts:
- added U1: ESP32-WROOM-32, RF_Module:ESP32-WROOM-32, symbol RF_Module:ESP32-WROOM-32
Connections:
- net GND: no longer SW1.C, SW1.S2
- new net: U1.1 (GND), U1.15 (GND), U1.38 (GND), U1.39 (GND)
Other:
- moved on the sheet: SW1
Changed lines of the file:
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@@
     (company "Ricardo Lima Caratti")
   )
-  (junction (at 119.38 48.26) (diameter 0) (color 0 0 0 0)
-  )
   (wire (pts (xy 158.75 48.26) (xy 170.18 48.26))
     (stroke (width 0) (type default))
   )
-  (wire (pts (xy 135.89 58.42) (xy 135.89 74.93))
+  (wire (pts (xy 116.84 66.04) (xy 116.84 67.31))
     (stroke (width 0) (type default))
   )
@@
     (stroke (width 0) (type default))
   )
-  (wire (pts (xy 114.3 49.53) (xy 114.3 12.7))
-    (stroke (width 0) (type default))
-  )
-  (wire (pts (xy 153.67 71.12) (xy 153.67 74.93))
-    (stroke (width 0) (type default))
-  )
-  (wire (pts (xy 146.05 68.58) (xy 146.05 74.93))
-    (stroke (width 0) (type default))
-  )
-  (wire (pts (xy 128.27 58.42) (xy 128.27 74.93))
-    (stroke (width 0) (type default))
-  )
-  (wire (pts (xy 148.59 58.42) (xy 148.59 68.58))
-    (stroke (width 0) (type default))
-  )
-  (wire (pts (xy 119.38 64.77) (xy 125.73 64.77))
-    (stroke (width 0) (type default))
-  )
   (wire (pts (xy 135.89 21.59) (xy 135.89 24.13))
     (stroke (width 0) (type default))
   )
-  (wire (pts (xy 133.35 58.42) (xy 133.35 74.93))
-    (stroke (width 0) (type default))
-  )
   (wire (pts (xy 149.86 24.13) (xy 158.75 24.13))
     (stroke (width 0) (type default))
   )
-  (wire (pts (xy 116.84 64.77) (xy 116.84 67.31))
-    (stroke (width 0) (type default))
-  )
-  (wire (pts (xy 123.19 72.39) (xy 114.3 72.39))
-    (stroke (width 0) (type default))
-  )
   (wire (pts (xy 146.05 27.94) (xy 146.05 38.1))
     (stroke (width 0) (type default))
@@
     (stroke (width 0) (type default))
   )
-  (wire (pts (xy 119.38 48.26) (xy 119.38 49.53))
+  (wire (pts (xy 86.36 48.26) (xy 86.36 49.53))
     (stroke (width 0) (type default))
   )
@@
     (stroke (width 0) (type default))
   )
-  (wire (pts (xy 153.67 66.04) (xy 153.67 58.42))
-    (stroke (width 0) (type default))
-  )
   (wire (pts (xy 127 34.29) (xy 133.35 34.29))
     (stroke (width 0) (type default))
@@
     (stroke (width 0) (type default))
   )
-  (wire (pts (xy 138.43 66.04) (xy 153.67 66.04))
-    (stroke (width 0) (type default))
-  )
   (wire (pts (xy 135.89 34.29) (xy 135.89 38.1))
     (stroke (width 0) (type default))
   )
-  (wire (pts (xy 123.19 74.93) (xy 123.19 72.39))
-    (stroke (width 0) (type default))
-  )
   (wire (pts (xy 142.24 24.13) (xy 135.89 24.13))
     (stroke (width 0) (type default))
   )
-  (wire (pts (xy 138.43 74.93) (xy 138.43 66.04))
-    (stroke (width 0) (type default))
-  )
-  (wire (pts (xy 176.53 12.7) (xy 176.53 71.12))
-    (stroke (width 0) (type default))
-  )
-  (wire (pts (xy 114.3 12.7) (xy 176.53 12.7))
-    (stroke (width 0) (type default))
-  )
-  (wire (pts (xy 125.73 74.93) (xy 125.73 64.77))
-    (stroke (width 0) (type default))
-  )
-  (wire (pts (xy 130.81 58.42) (xy 130.81 74.93))
-    (stroke (width 0) (type default))
-  )
-  (wire (pts (xy 176.53 71.12) (xy 153.67 71.12))
-    (stroke (width 0) (type default))
-  )
-  (wire (pts (xy 114.3 72.39) (xy 114.3 64.77))
-    (stroke (width 0) (type default))
-  )
   (wire (pts (xy 133.35 38.1) (xy 133.35 34.29))
     (stroke (width 0) (type default))
   )
   (wire (pts (xy 170.18 48.26) (xy 170.18 46.99))
-    (stroke (width 0) (type default))
-  )
-  (wire (pts (xy 148.59 68.58) (xy 146.05 68.58))
     (stroke (width 0) (type default))
   )
@@
     )
   )
-  (symbol (lib_id "Device:RotaryEncoder_Switch") (at 116.84 57.15 90) (unit 1)
-    (in_bom yes) (on_board yes) (dnp no)
-    (property "Reference" "SW1" (at 104.14 52.07 90)
+  (symbol (lib_id "Device:RotaryEncoder_Switch") (at 83.82 57.15 90) (unit 1)
+    (in_bom yes) (on_board yes) (dnp no)
+    (property "Reference" "SW1" (at 71.12 52.07 90)
       (effects (font (size 1.27 1.27)) (justify right))
     )
-    (property "Value" "ENCODER" (at 101.6 54.61 90)
+    (property "Value" "ENCODER" (at 68.58 54.61 90)
       (effects (font (size 1.27 1.27)) (justify right))
     )
-    (property "Footprint" "" (at 112.776 60.96 0)
-      (effects (font (size 1.27 1.27)) hide)
-    )
-    (property "Datasheet" "~" (at 110.236 57.15 0)
+    (property "Footprint" "" (at 79.756 60.96 0)
+      (effects (font (size 1.27 1.27)) hide)
+    )
+    (property "Datasheet" "~" (at 77.216 57.15 0)
       (effects (font (size 1.27 1.27)) hide)
     )
@@
         )
       )
+    )
+  )
+  (symbol (lib_id "RF_Module:ESP32-WROOM-32") (at 41.91 81.28 0) (unit 1)
+    (in_bom yes) (on_board yes) (dnp no) (fields_autoplaced)
+    (property "Reference" "U1" (at 43.8659 43.18 0)
+      (effects (font (size 1.27 1.27)) (justify left))
+    )
+    (property "Value" "ESP32-WROOM-32" (at 43.8659 45.72 0)
+      (effects (font (size 1.27 1.27)) (justify left))
+    )
+    (property "Footprint" "RF_Module:ESP32-WROOM-32" (at 41.91 119.38 0)
+      (effects (font (size 1.27 1.27)) hide)
+    )
+    (property "Datasheet" "https://www.espressif.com/sites/default/files/documentation/esp32-wroom-32_datasheet_en.pdf" (at 34.29 80.01 0)
+      (effects (font (size 1.27 1.27)) hide)
+    )
+    (pin "1")
+    (pin "10")
+    (pin "11")
+    (pin "12")
+    (pin "13")
+    (pin "14")
+    (pin "15")
+    (pin "16")
+    (pin "17")
+    (pin "18")
+    (pin "19")
+    (pin "2")
+    (pin "20")
+    (pin "21")
+    (pin "22")
+    (pin "23")
+    (pin "24")
+    (pin "25")
+    (pin "26")
+    (pin "27")
+    (pin "28")
+    (pin "29")
+    (pin "3")
+    (pin "30")
+    (pin "31")
+    (pin "32")
+    (pin "33")
+    (pin "34")
+    (pin "35")
+    (pin "36")
+    (pin "37")
+    (pin "38")
+    (pin "39")
+    (pin "4")
+    (pin "5")
+    (pin "6")
+    (pin "7")
+    (pin "8")
+    (pin "9")
+    (instances
+      (project "ESP32_LCD_ENCODER"
+        (path "/88d7f29c-c2c1-4d72-a8c4-9ed549acb450"
+          (reference "U1") (unit 1)
+        )
+      )
