File: examples/03_TX_LCD_16x2_AND_20x4/KiCad_Schematic/STANDALONE_ATMEGA328/schematic_basic_atmega328_standalone_12MHz_LCD16x2.kicad_sch (KiCad schematic)
At the start: 11 parts, among them J1 QN8066, J2 Power Control / PWM, U2 ATMEGA328P_PDIP, Y1 12MHz

Commit message: Doc
Parts:
- added J3: AVR-ISP-6, symbol Connector:AVR-ISP-6
- added J4: PC6/RESET, symbol Connector:Conn_01x01_Pin
Connections:
- net +3.3VP: now also J3.2 (VCC)
- net GND: now also J3.6 (GND)
- net at LCD1.4 (RS), LCD2.4 (RS), U2.18 (PB4(MISO)): now also J3.1 (MISO)
- net at LCD1.6 (E), LCD2.6 (E), U2.19 (PB5(SCK)): now also J3.3 (SCK)
- net at U2.17 (PB3(MOSI/OC2)): now also J3.4 (MOSI)
- new net: J3.5 (~{RST}), J4.1 (Pin_1)
Changed lines of the file:
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@@
   (junction (at 128.27 45.72) (diameter 0) (color 0 0 0 0)
   )
+  (junction (at 149.86 132.08) (diameter 0) (color 0 0 0 0)
+  )
   (junction (at 161.29 45.72) (diameter 0) (color 0 0 0 0)
   )
@@
   (junction (at 158.75 45.72) (diameter 0) (color 0 0 0 0)
   )
+  (junction (at 144.78 129.54) (diameter 0) (color 0 0 0 0)
+  )
   (junction (at 107.95 49.53) (diameter 0) (color 0 0 0 0)
   )
   (junction (at 228.6 101.6) (diameter 0) (color 0 0 0 0)
   )
-  (wire (pts (xy 138.43 132.08) (xy 151.13 132.08))
+  (wire (pts (xy 138.43 132.08) (xy 149.86 132.08))
     (stroke (width 0.1524) (type solid))
   )
@@
     (stroke (width 0.1524) (type solid))
   )
+  (wire (pts (xy 152.4 148.59) (xy 152.4 147.32))
+    (stroke (width 0) (type default))
+  )
   (wire (pts (xy 87.63 93.98) (xy 87.63 73.66))
     (stroke (width 0.1524) (type solid))
@@
     (stroke (width 0) (type default))
   )
+  (wire (pts (xy 144.78 129.54) (xy 144.78 148.59))
+    (stroke (width 0) (type default))
+  )
   (wire (pts (xy 161.29 66.04) (xy 148.59 66.04))
     (stroke (width 0.1524) (type solid))
@@
     (stroke (width 0.1524) (type solid))
   )
+  (wire (pts (xy 144.78 129.54) (xy 135.89 129.54))
+    (stroke (width 0.1524) (type solid))
+  )
   (wire (pts (xy 118.11 68.58) (xy 107.95 68.58))
     (stroke (width 0) (type default))
   )
+  (wire (pts (xy 149.86 132.08) (xy 149.86 148.59))
+    (stroke (width 0) (type default))
+  )
   (wire (pts (xy 163.83 58.42) (xy 199.39 58.42))
     (stroke (width 0.1524) (type solid))
@@
     (stroke (width 0) (type default))
   )
+  (wire (pts (xy 160.02 161.29) (xy 161.29 161.29))
+    (stroke (width 0) (type default))
+  )
   (wire (pts (xy 101.6 49.53) (xy 107.95 49.53))
     (stroke (width 0) (type default))
@@
     (stroke (width 0) (type default))
   )
-  (wire (pts (xy 151.13 129.54) (xy 135.89 129.54))
+  (wire (pts (xy 151.13 129.54) (xy 144.78 129.54))
     (stroke (width 0.1524) (type solid))
   )
@@
     (stroke (width 0) (type default))
   )
+  (wire (pts (xy 149.86 132.08) (xy 151.13 132.08))
+    (stroke (width 0.1524) (type solid))
+  )
   (wire (pts (xy 69.85 83.82) (xy 74.93 83.82))
     (stroke (width 0) (type default))
@@
     (stroke (width 0.1524) (type solid))
   )
+  (wire (pts (xy 137.16 161.29) (xy 134.62 161.29))
+    (stroke (width 0) (type default))
+  )
   (wire (pts (xy 97.79 109.22) (xy 97.79 113.03))
     (stroke (width 0) (type default))
@@
     (stroke (width 0) (type default))
   )
+  (wire (pts (xy 147.32 127) (xy 151.13 127))
+    (stroke (width 0) (type default))
+  )
+  (wire (pts (xy 152.4 147.32) (xy 160.02 147.32))
+    (stroke (width 0) (type default))
+  )
   (wire (pts (xy 233.68 129.54) (xy 233.68 132.08))
     (stroke (width 0.1524) (type solid))
@@
     (stroke (width 0) (type default))
   )
+  (wire (pts (xy 161.29 161.29) (xy 161.29 165.1))
+    (stroke (width 0) (type default))
+  )
   (wire (pts (xy 69.85 86.36) (xy 151.13 86.36))
     (stroke (width 0) (type default))
@@
     (stroke (width 0) (type default))
   )
+  (wire (pts (xy 147.32 148.59) (xy 147.32 127))
+    (stroke (width 0) (type default))
+  )
   (wire (pts (xy 133.35 45.72) (xy 133.35 59.69))
     (stroke (width 0) (type default))
@@
   )
   (wire (pts (xy 118.11 45.72) (xy 128.27 45.72))
+    (stroke (width 0) (type default))
+  )
+  (wire (pts (xy 134.62 161.29) (xy 134.62 158.75))
     (stroke (width 0) (type default))
   )
@@
     (effects (font (size 1.778 1.5113)) (justify left bottom))
   )
-  (text "D13" (at 140.97 134.62 0)
+  (text "D13" (at 138.43 134.62 0)
     (effects (font (size 1.778 1.5113)) (justify left bottom))
   )
@@
   (text "SCL" (at 72.39 88.9 0)
     (effects (font (size 1.27 1.27)) (justify left bottom))
+  )
+  (symbol (lib_id "Connector:AVR-ISP-6") (at 149.86 158.75 90) (unit 1)
+    (in_bom yes) (on_board yes) (dnp no) (fields_autoplaced)
+    (property "Reference" "J3" (at 148.59 168.91 90)
+      (effects (font (size 1.27 1.27)))
+    )
+    (property "Value" "AVR-ISP-6" (at 148.59 171.45 90)
+      (effects (font (size 1.27 1.27)))
+    )
+    (property "Footprint" "" (at 148.59 165.1 90)
+      (effects (font (size 1.27 1.27)) hide)
+    )
+    (property "Datasheet" " ~" (at 163.83 191.135 0)
+      (effects (font (size 1.27 1.27)) hide)
+    )
+    (pin "1")
+    (pin "2")
+    (pin "3")
+    (pin "4")
+    (pin "5")
+    (pin "6")
+    (instances
+      (project "schematic_basic_atmega328_standalone_12MHz_LCD16x2"
+        (path "/88d7f29c-c2c1-4d72-a8c4-9ed549acb450"
+          (reference "J3") (unit 1)
+        )
+      )
+    )
   )
   (symbol (lib_id "schematic_basic_atmega328_standalone_12MHz_LCD16x2-eagle-import:LCD-16X2SILK") (at 148.59 35.56 90) (unit 1)
@@
         (path "/88d7f29c-c2c1-4d72-a8c4-9ed549acb450"
           (reference "#PWR02") (unit 1)
+        )
+      )
+    )
+  )
+  (symbol (lib_id "Connector:Conn_01x01_Pin") (at 165.1 147.32 180) (unit 1)
+    (in_bom yes) (on_board yes) (dnp no) (fields_autoplaced)
+    (property "Reference" "J4" (at 164.465 142.24 0)
+      (effects (font (size 1.27 1.27)))
+    )
+    (property "Value" "PC6/RESET" (at 164.465 144.78 0)
+      (effects (font (size 1.27 1.27)))
+    )
+    (property "Footprint" "" (at 165.1 147.32 0)
+      (effects (font (size 1.27 1.27)) hide)
+    )
+    (property "Datasheet" "~" (at 165.1 147.32 0)
+      (effects (font (size 1.27 1.27)) hide)
+    )
+    (pin "1")
+    (instances
+      (project "schematic_basic_atmega328_standalone_12MHz_LCD16x2"
+        (path "/88d7f29c-c2c1-4d72-a8c4-9ed549acb450"
+          (reference "J4") (unit 1)
         )
       )
@@
     )
   )
+  (symbol (lib_id "power:GND") (at 161.29 165.1 0) (unit 1)
+    (in_bom yes) (on_board yes) (dnp no) (fields_autoplaced)
+    (property "Reference" "#PWR010" (at 161.29 171.45 0)
+      (effects (font (size 1.27 1.27)) hide)
+    )
+    (property "Value" "GND" (at 161.29 170.18 0)
+      (effects (font (size 1.27 1.27)))
+    )
+    (property "Footprint" "" (at 161.29 165.1 0)
+      (effects (font (size 1.27 1.27)) hide)
+    )
+    (property "Datasheet" "" (at 161.29 165.1 0)
+      (effects (font (size 1.27 1.27)) hide)
+    )
+    (pin "1")
+    (instances
+      (project "schematic_basic_atmega328_standalone_12MHz_LCD16x2"
+        (path "/88d7f29c-c2c1-4d72-a8c4-9ed549acb450"
+          (reference "#PWR010") (unit 1)
+        )
+      )
+    )
+  )
   (symbol (lib_id "power:GND") (at 57.15 104.14 0) (unit 1)
     (in_bom yes) (on_board yes) (dnp no) (fields_autoplaced)
@@
         )
       )
+    )
+  )
+  (symbol (lib_id "power:+3.3VP") (at 134.62 158.75 0) (unit 1)
+    (in_bom yes) (on_board yes) (dnp no) (fields_autoplaced)
+    (property "Reference" "#PWR011" (at 138.43 160.02 0)
+      (effects (font (size 1.27 1.27)) hide)
+    )
+    (property "Value" "+3.3VP" (at 134.62 153.67 0)
+      (effects (font (size 1.27 1.27)))
+    )
+    (property "Footprint" "" (at 134.62 158.75 0)
+      (effects (font (size 1.27 1.27)) hide)
+    )
+    (property "Datasheet" "" (at 134.62 158.75 0)
+      (effects (font (size 1.27 1.27)) hide)
+    )
+    (pin "1")
+    (instances
+      (project "schematic_basic_atmega328_standalone_12MHz_LCD16x2"
+        (path "/88d7f29c-c2c1-4d72-a8c4-9ed549acb450"
+          (reference "#PWR011") (unit 1)
+        )
+      )

Commit message: Doc
Connections:
- net at S2.SW+: now also U2.14 (PB0(ICP)); no longer U2.23 (PC0(ADC0))
Other:
- note added: "D8"
- moved on the sheet: C1, C2, J1, J2, J3, J4, R1, RV1, S2, U2, Y1
