File: examples/03_TX_LCD_16x2_AND_20x4/03_ESP32/KiCad/ESP32_LCD_ENCODER/ESP32_LCD_ENCODER.kicad_sch (KiCad schematic)
At the start: 5 parts, among them SW1 ENCODER, U1 ESP32-WROOM-32, U2 LCD16X2

Commit message: Doc
Connections:
- net +3.3V: now also U1.2 (VDD)
Other:
- moved on the sheet: QN1, RV1, SW1, U1, U2
