File: examples/07_WEB_WIFI_ESP32_QN8066/KiCad/ESP32_WEB/ESP32_WEB.kicad_sch (KiCad schematic)
At the start: 3 parts, among them J1 PWM, U1 ESP32-WROOM-32

Commit message: Doc
Parts:
- added C1, C2: 1uF, symbol Device:C
- added J2: Audio In, symbol Connector_Audio:AudioJack2_Ground
- added R1, R2: 4.7K, symbol Device:R
- added R3, R4: 10K, symbol Device:R
Connections:
- net +3.3V: now also QN1.13 (CEN), QN1.3 (VCC), R1.2, R2.2
- net GND: now also QN1.11 (GND), QN1.15 (GND), QN1.6 (GND), R3.2, R4.2
- net at QN1.1 (SCL), U1.36 (IO22): now also R1.1
- net at QN1.10 (ALI): now also C1.1, R4.1
- net at QN1.2 (SCA), U1.33 (IO21): now also R2.1
- net at QN1.9 (ARI): now also C2.1, R3.1
- new net: C2.2, J2.T
- new net: C1.2, J2.S
