File: examples/07_ESP32/01_ESP32_LCD16x2_ENCODER/KiCad/ESP32_LCD_ENCODER/ESP32_LCD_ENCODER.kicad_sch (KiCad schematic)
At the start: 5 parts, among them SW1 ENCODER, U1 ESP32-WROOM-32, U2 LCD16X2

Commit message: Doc
Parts:
- added AE1: Antenna, symbol Device:Antenna
- added C1: 15pF, symbol Device:C
- added C2, C3: 1uF, symbol Device:C
- added J1: AudioJack2_Ground, symbol Connector_Audio:AudioJack2_Ground
- added L1: 150nH, symbol Device:L
- added R1, R2: 150R, symbol Device:R
- added R3, R4: 4.7K, symbol Device:R
- added X1: 32.768MHz, Oscillator:Oscillator_DIP-14, symbol Oscillator:ACO-xxxMHz
Connections:
- net +3.3V: now also QN1.13 (CEN), QN1.3 (VCC), R3.1, R4.1, X1.14 (Vcc)
- net GND: now also QN1.11 (GND), QN1.15 (GND), QN1.6 (GND), J1.G, L1.1, X1.7 (GND)
- net at QN1.1 (SCL): now also R1.2, R3.2; no longer U1.36 (IO22)
- net at QN1.10 (ALI): now also C2.2
- net at QN1.12 (RFO): now also C1.2, L1.2
- net at QN1.14 (XCLC): now also X1.8 (OUT)
- net at QN1.2 (SCA): now also R2.2, R4.2; no longer U1.33 (IO21)
- net at QN1.9 (ARI): now also C3.2
- new net: R2.1, U1.33 (IO21)
- new net: C3.1, J1.S
- new net: C2.1, J1.T
- new net: AE1.1 (A), C1.1
- new net: R1.1, U1.36 (IO22)
Other:
- note added: "32.768MHz"
- note added: "Active Crystal"
- moved on the sheet: QN1, RV1, SW1, U1, U2
