File: examples/08_STM32/KiCad/STM32_LCD_ENCODER/STM32_LCD_ENCODER.kicad_sch (KiCad schematic)
At the start: 17 parts, among them J1 Audio In, SW1 ENCODER, U1 STM32F103C6Tx, U2 LCD16X2

Commit message: Doc
Parts:
- added X1: ACO-32.768MHz, Oscillator:Oscillator_DIP-14, symbol Oscillator:ACO-xxxMHz
Connections:
- net +3.3V: now also QN1.13 (CEN), X1.14 (Vcc)
- net GND: now also X1.7 (GND)
- net at QN1.14 (XCLC): now also X1.8 (OUT)
Changed lines of the file:
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@@
 (kicad_sch (version 20230121) (generator eeschema)
-  (paper "User" 200 200)
+  (paper "User" 219.989 219.989)
   (title_block
     (title "STM32 WITH  LCD16x2, ENCODER AND QN8066")
@@
   (junction (at 102.87 137.16) (diameter 0) (color 0 0 0 0)
   )
+  (junction (at 69.85 110.49) (diameter 0) (color 0 0 0 0)
+  )
   (junction (at 55.88 146.05) (diameter 0) (color 0 0 0 0)
   )
@@
   (junction (at 53.34 129.54) (diameter 0) (color 0 0 0 0)
   )
-  (junction (at 67.31 110.49) (diameter 0) (color 0 0 0 0)
-  )
   (junction (at 58.42 137.16) (diameter 0) (color 0 0 0 0)
   )
@@
     (stroke (width 0) (type default))
   )
+  (wire (pts (xy 68.58 154.94) (xy 68.58 158.75))
+    (stroke (width 0) (type default))
+  )
   (wire (pts (xy 81.28 31.75) (xy 87.63 31.75))
     (stroke (width 0) (type default))
   )
+  (wire (pts (xy 87.63 158.75) (xy 91.44 158.75))
+    (stroke (width 0) (type default))
+  )
+  (wire (pts (xy 72.39 158.75) (xy 68.58 158.75))
+    (stroke (width 0) (type default))
+  )
   (wire (pts (xy 67.31 110.49) (xy 67.31 111.76))
     (stroke (width 0) (type default))
@@
     (stroke (width 0) (type default))
   )
-  (wire (pts (xy 80.01 106.68) (xy 52.07 106.68))
-    (stroke (width 0) (type default))
-  )
   (wire (pts (xy 101.6 109.22) (xy 101.6 110.49))
     (stroke (width 0) (type default))
@@
     (stroke (width 0) (type default))
   )
+  (wire (pts (xy 77.47 128.27) (xy 77.47 130.81))
+    (stroke (width 0) (type default))
+  )
   (wire (pts (xy 85.09 97.79) (xy 85.09 100.33))
     (stroke (width 0) (type default))
   )
-  (wire (pts (xy 80.01 111.76) (xy 80.01 106.68))
-    (stroke (width 0) (type default))
-  )
   (wire (pts (xy 81.28 34.29) (xy 81.28 31.75))
     (stroke (width 0) (type default))
@@
     (stroke (width 0) (type default))
   )
-  (wire (pts (xy 52.07 110.49) (xy 67.31 110.49))
+  (wire (pts (xy 91.44 158.75) (xy 91.44 161.29))
     (stroke (width 0) (type default))
   )
@@
     (stroke (width 0) (type default))
   )
-  (wire (pts (xy 52.07 102.87) (xy 52.07 106.68))
-    (stroke (width 0) (type default))
-  )
   (wire (pts (xy 105.41 49.53) (xy 105.41 64.77))
     (stroke (width 0) (type default))
@@
     (stroke (width 0) (type default))
   )
+  (wire (pts (xy 80.01 107.95) (xy 80.01 111.76))
+    (stroke (width 0) (type default))
+  )
   (wire (pts (xy 74.93 137.16) (xy 102.87 137.16))
     (stroke (width 0) (type default))
@@
     (stroke (width 0) (type default))
   )
-  (wire (pts (xy 72.39 110.49) (xy 67.31 110.49))
+  (wire (pts (xy 72.39 110.49) (xy 69.85 110.49))
     (stroke (width 0) (type default))
   )
@@
     (stroke (width 0) (type default))
   )
+  (wire (pts (xy 80.01 128.27) (xy 80.01 151.13))
+    (stroke (width 0) (type default))
+  )
   (wire (pts (xy 124.46 22.86) (xy 118.11 22.86))
     (stroke (width 0) (type default))
@@
   )
   (wire (pts (xy 35.56 132.08) (xy 40.64 132.08))
+    (stroke (width 0) (type default))
+  )
+  (wire (pts (xy 69.85 110.49) (xy 67.31 110.49))
+    (stroke (width 0) (type default))
+  )
+  (wire (pts (xy 69.85 107.95) (xy 69.85 110.49))
     (stroke (width 0) (type default))
   )
@@
         (path "/88d7f29c-c2c1-4d72-a8c4-9ed549acb450"
           (reference "R2") (unit 1)
+        )
+      )
+    )
+  )
+  (symbol (lib_id "Oscillator:ACO-xxxMHz") (at 80.01 158.75 90) (unit 1)
+    (in_bom yes) (on_board yes) (dnp no) (fields_autoplaced)
+    (property "Reference" "X1" (at 80.01 166.37 90)
+      (effects (font (size 1.27 1.27)))
+    )
+    (property "Value" "ACO-32.768MHz" (at 80.01 168.91 90)
+      (effects (font (size 1.27 1.27)))
+    )
+    (property "Footprint" "Oscillator:Oscillator_DIP-14" (at 88.9 147.32 0)
+      (effects (font (size 1.27 1.27)) hide)
+    )
+    (property "Datasheet" "http://www.conwin.com/datasheets/cx/cx030.pdf" (at 80.01 161.29 0)
+      (effects (font (size 1.27 1.27)) hide)
+    )
+    (pin "1")
+    (pin "14")
+    (pin "7")
+    (pin "8")
+    (instances
+      (project "STM32_LCD_ENCODER"
+        (path "/88d7f29c-c2c1-4d72-a8c4-9ed549acb450"
+          (reference "X1") (unit 1)
         )
       )
@@
   (symbol (lib_id "Device:R") (at 82.55 104.14 0) (mirror y) (unit 1)
     (in_bom yes) (on_board yes) (dnp no)
-    (property "Reference" "R3" (at 80.01 102.87 0)
+    (property "Reference" "R3" (at 81.28 100.33 0)
       (effects (font (size 1.27 1.27)) (justify left))
     )
-    (property "Value" "150R" (at 80.01 105.41 0)
+    (property "Value" "150R" (at 80.01 102.87 0)
       (effects (font (size 1.27 1.27)) (justify left))
     )
@@
     )
   )
-  (symbol (lib_id "power:+3.3V") (at 52.07 102.87 0) (unit 1)
-    (in_bom yes) (on_board yes) (dnp no) (fields_autoplaced)
-    (property "Reference" "#PWR013" (at 52.07 106.68 0)
-      (effects (font (size 1.27 1.27)) hide)
-    )
-    (property "Value" "+3.3V" (at 52.07 97.79 0)
-      (effects (font (size 1.27 1.27)))
-    )
-    (property "Footprint" "" (at 52.07 102.87 0)
-      (effects (font (size 1.27 1.27)) hide)
-    )
-    (property "Datasheet" "" (at 52.07 102.87 0)
+  (symbol (lib_id "power:+3.3V") (at 80.01 107.95 0) (unit 1)
+    (in_bom yes) (on_board yes) (dnp no)
+    (property "Reference" "#PWR013" (at 80.01 111.76 0)
+      (effects (font (size 1.27 1.27)) hide)
+    )
+    (property "Value" "+3.3V" (at 76.2 106.68 0)
+      (effects (font (size 1.27 1.27)))
+    )
+    (property "Footprint" "" (at 80.01 107.95 0)
+      (effects (font (size 1.27 1.27)) hide)
+    )
+    (property "Datasheet" "" (at 80.01 107.95 0)
       (effects (font (size 1.27 1.27)) hide)
     )
@@
     )
   )
-  (symbol (lib_id "power:GND") (at 52.07 110.49 0) (unit 1)
-    (in_bom yes) (on_board yes) (dnp no)
-    (property "Reference" "#PWR012" (at 52.07 116.84 0)
-      (effects (font (size 1.27 1.27)) hide)
-    )
-    (property "Value" "GND" (at 52.07 114.3 0)
-      (effects (font (size 1.27 1.27)))
-    )
-    (property "Footprint" "" (at 52.07 110.49 0)
-      (effects (font (size 1.27 1.27)) hide)
-    )
-    (property "Datasheet" "" (at 52.07 110.49 0)
+  (symbol (lib_id "power:GND") (at 69.85 107.95 180) (unit 1)
+    (in_bom yes) (on_board yes) (dnp no)
+    (property "Reference" "#PWR012" (at 69.85 101.6 0)
+      (effects (font (size 1.27 1.27)) hide)
+    )
+    (property "Value" "GND" (at 69.85 104.14 0)
+      (effects (font (size 1.27 1.27)))
+    )
+    (property "Footprint" "" (at 69.85 107.95 0)
+      (effects (font (size 1.27 1.27)) hide)
+    )
+    (property "Datasheet" "" (at 69.85 107.95 0)
       (effects (font (size 1.27 1.27)) hide)
     )
@@
     )
   )
+  (symbol (lib_id "power:GND") (at 91.44 161.29 0) (unit 1)
+    (in_bom yes) (on_board yes) (dnp no)
+    (property "Reference" "#PWR020" (at 91.44 167.64 0)
+      (effects (font (size 1.27 1.27)) hide)
+    )
+    (property "Value" "GND" (at 91.44 165.1 0)
+      (effects (font (size 1.27 1.27)))
+    )
+    (property "Footprint" "" (at 91.44 161.29 0)
+      (effects (font (size 1.27 1.27)) hide)
+    )
+    (property "Datasheet" "" (at 91.44 161.29 0)
+      (effects (font (size 1.27 1.27)) hide)
+    )
+    (pin "1")
+    (instances
+      (project "STM32_LCD_ENCODER"
+        (path "/88d7f29c-c2c1-4d72-a8c4-9ed549acb450"
+          (reference "#PWR020") (unit 1)
+        )
+      )
+    )
+  )
   (symbol (lib_id "power:+3.3V") (at 149.86 80.01 0) (unit 1)
     (in_bom yes) (on_board yes) (dnp no) (fields_autoplaced)
@@
         (path "/88d7f29c-c2c1-4d72-a8c4-9ed549acb450"
           (reference "#PWR011") (unit 1)
+        )
+      )
+    )
+  )
+  (symbol (lib_id "power:+3.3V") (at 68.58 154.94 0) (unit 1)
+    (in_bom yes) (on_board yes) (dnp no) (fields_autoplaced)
+    (property "Reference" "#PWR021" (at 68.58 158.75 0)
+      (effects (font (size 1.27 1.27)) hide)
+    )
+    (property "Value" "+3.3V" (at 68.58 149.86 0)
+      (effects (font (size 1.27 1.27)))
+    )
+    (property "Footprint" "" (at 68.58 154.94 0)
+      (effects (font (size 1.27 1.27)) hide)
+    )
+    (property "Datasheet" "" (at 68.58 154.94 0)
+      (effects (font (size 1.27 1.27)) hide)
+    )
+    (pin "1")
+    (instances
+      (project "STM32_LCD_ENCODER"
+        (path "/88d7f29c-c2c1-4d72-a8c4-9ed549acb450"
+          (reference "#PWR021") (unit 1)
         )
       )
@@
   (symbol (lib_id "Device:R") (at 85.09 104.14 0) (unit 1)
     (in_bom yes) (on_board yes) (dnp no)
-    (property "Reference" "R4" (at 87.63 102.87 0)
+    (property "Reference" "R4" (at 87.63 100.33 0)
       (effects (font (size 1.27 1.27)) (justify left))
     )
-    (property "Value" "150R" (at 87.63 105.41 0)
+    (property "Value" "150R" (at 87.63 102.87 0)
       (effects (font (size 1.27 1.27)) (justify left))
     )
@@
         )
       )
+    )
+  )
+  (symbol (lib_id "power:+3.3V") (at 77.47 130.81 180) (unit 1)
+    (in_bom yes) (on_board yes) (dnp no)
+    (property "Reference" "#PWR022" (at 77.47 127 0)
+      (effects (font (size 1.27 1.27)) hide)
+    )
+    (property "Value" "+3.3V" (at 77.47 137.16 90)
+      (effects (font (size 1.27 1.27)) hide)
+    )
+    (property "Footprint" "" (at 77.47 130.81 0)
+      (effects (font (size 1.27 1.27)) hide)
+    )
+    (property "Datasheet" "" (at 77.47 130.81 0)
+      (effects (font (size 1.27 1.27)) hide)
+    )
+    (pin "1")
+    (instances
+      (project "STM32_LCD_ENCODER"
+        (path "/88d7f29c-c2c1-4d72-a8c4-9ed549acb450"
+          (reference "#PWR022") (unit 1)
+        )
+      )

Commit message: Doc
Parts:
- added C4, C5: 10pF, symbol Device:C
- added RTC: 32.768kHz, symbol Device:Crystal
- added RTC_BAT: 3V, symbol Device:Battery
Connections:
- net GND: now also C4.2, C5.2, RTC_BAT.2 (-)
- net at U1.1 (VBAT): now also RTC_BAT.1 (+)
- net at U1.3 (PC14): now also C4.1, RTC.1
- net at U1.4 (PC15): now also C5.1, RTC.2
Other:
- note added: "Optional"
- moved on the sheet: R5, R6
