File: extras/schematics/Small_RF_AMP/Small_RF_AMP.kicad_sch (KiCad schematic)
At the start: 12 parts, among them J1 RF Input

Commit message: Doc
Parts:
- added C6: 62pF, symbol Device:C
- C1: value 22pF -> 100pF
- L1: value 150nF -> 62nF
- L2: value 47nF -> ??nF
Connections:
- net GND: now also C6.2; no longer L1.2
- net at R1.2, S9018.2 (B): now also L1.2; no longer C1.1
- net at C1.2, J1.1 (In): no longer L1.1
- new net: C1.1, C6.1, L1.1
Other:
- moved on the sheet: AE1, C1, C2, C3, C4, C5, J1, L2, R1, R2, S9018

Commit message: Doc
Parts:
- added C3: 33pF, symbol Device:C
- added L2: 6.2nF, symbol Device:L
- C2: renamed from C6; value 62pF -> 100pF
- renumbered C3 to C4, C2 to C6, C5 to C7, C4 to C8, L2 to L3
Connections:
- net GND: now also L2.1
- net at R1.2, S9018.2 (B): now also C3.1; no longer L1.2
- new net: C3.2, L1.2, L2.2
Other:
- moved on the sheet: AE1, C2, C4, C6, C7, C8, L3, R1, R2, S9018

Commit message: Doc
Parts:
- L2: value 6.2nF -> 6.5nF
Changed lines of the file:
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@@
       (effects (font (size 1.27 1.27)) (justify right))
     )
-    (property "Value" "6.2nF" (at 66.04 76.2 0)
+    (property "Value" "6.5nF" (at 66.04 76.2 0)
       (effects (font (size 1.27 1.27)) (justify right))
     )
